Commit message: Update robot description package with latest changes

File: urdf/robot.urdf.xacro (robot description, xacro)
@@ -1,4 +1,5 @@
 <?xml version="1.0"?>
 <robot name="my_robot" xmlns:xacro="http://www.ros.org/wiki/xacro">
+    <xacro:include filename="$(find my_robot_description)/urdf/robot.gazebo.xacro"/>
     <xacro:property name="base_length" value="0.3"/>
     <xacro:property name="base_width"  value="0.3"/>
@@ -15,4 +16,5 @@
     <xacro:property name="lidar_mass"   value="0.1"/>
     <xacro:property name="lidar_z_offset" value="0.13"/>
+    <xacro:property name="mesh_path" default="package://my_robot_description/meshes"/>
     <xacro:property name="base_footprint_z" value="0.15"/>
     <link name="base_footprint"/>
@@ -43,5 +45,5 @@
     <link name="lidar_link">
         <visual>
-            <geometry><cylinder radius="${lidar_radius}" length="${lidar_length}"/></geometry>
+            <geometry><mesh filename="$(mesh_path)lidar.STL"/></geometry>
             <material name="lidar_gray"><color rgba="0.5 0.5 0.5 1.0"/></material>
         </visual>
@@ -91,73 +93,3 @@
     <xacro:wheel prefix="left_back"   x_reflect="-1" y_reflect="1"/>
     <xacro:wheel prefix="right_back"  x_reflect="-1" y_reflect="-1"/>
-    <gazebo>
-        <plugin name="gz::sim::systems::DiffDrive" filename="gz-sim-diff-drive-system">
-            <left_joint>left_front_wheel_joint</left_joint>
-            <right_joint>right_front_wheel_joint</right_joint>
-            <wheel_separation>${2 * wheel_y_offset}</wheel_separation>
-            <wheel_diameter>${2 * wheel_radius}</wheel_diameter>
-            <topic>/cmd_vel</topic>
-            <odom_frame>odom</odom_frame>
-            <robot_base_frame>base_footprint</robot_base_frame>
-            <publish_odom>true</publish_odom>
-            <publish_odom_tf>true</publish_odom_tf>
-            <update_rate>50</update_rate>
-            <max_linear_velocity>0.5</max_linear_velocity>
-            <min_linear_velocity>-0.5</min_linear_velocity>
-            <max_angular_velocity>1.0</max_angular_velocity>
-            <min_angular_velocity>-1.0</min_angular_velocity>
-            <max_linear_acceleration>1.0</max_linear_acceleration>
-            <min_linear_acceleration>-1.0</min_linear_acceleration>
-            <max_angular_acceleration>2.0</max_angular_acceleration>
-            <min_angular_acceleration>-2.0</min_angular_acceleration>
-        </plugin>
-    </gazebo>
-    <gazebo>
-        <plugin name="gz::sim::systems::JointStatePublisher" filename="gz-sim-joint-state-publisher-system">
-            <joint_name>left_front_wheel_joint</joint_name>
-            <joint_name>left_back_wheel_joint</joint_name>
-            <joint_name>right_front_wheel_joint</joint_name>
-            <joint_name>right_back_wheel_joint</joint_name>
-            <update_rate>30</update_rate>
-        </plugin>
-    </gazebo>
-    <gazebo>
-        <plugin name="gz::sim::systems::OdometryPublisher" filename="gz-sim-odometry-publisher-system">
-            <odom_frame>odom</odom_frame>
-            <robot_base_frame>base_footprint</robot_base_frame>
-            <odom_topic>odom</odom_topic>
-            <tf_topic>/tf</tf_topic>
-            <odom_publish_frequency>50</odom_publish_frequency>
-        </plugin>
-    </gazebo>
-    <gazebo reference="lidar_link">
-        <sensor name="lidar_sensor" type="gpu_lidar">
-            <topic>/scan</topic>
-            <update_rate>30</update_rate>
-            <gz_frame_id>lidar_link</gz_frame_id>
-            <lidar>
-                <scan>
-                    <horizontal>
-                        <samples>720</samples>
-                        <resolution>1</resolution>
-                        <min_angle>-3.14</min_angle>
-                        <max_angle>3.14</max_angle>
-                    </horizontal>
-                    <vertical>
-                        <samples>1</samples>
-                        <resolution>1</resolution>
-                        <min_angle>0</min_angle>
-                        <max_angle>0</max_angle>
-                    </vertical>
-                </scan>
-                <range>
-                    <min>0.15</min>
-                    <max>10.0</max>
-                    <resolution>0.01</resolution>
-                </range>
-            </lidar>
-            <always_on>true</always_on>
-            <visualize>true</visualize>
-        </sensor>
-    </gazebo>
 </robot>
