Commit message: Update robot description files

File: my_robot_description/urdf/robot.gazebo.xacro (robot description, xacro)
@@ -6,5 +6,7 @@
         <plugin name="gz::sim::systems::DiffDrive" filename="gz-sim-diff-drive-system">
             <left_joint>left_front_wheel_joint</left_joint>
+            <left_joint>left_back_wheel_joint</left_joint>
             <right_joint>right_front_wheel_joint</right_joint>
+            <right_joint>right_back_wheel_joint</right_joint>
             <wheel_separation>${2 * wheel_y_offset}</wheel_separation>
             <wheel_diameter>${2 * wheel_radius}</wheel_diameter>

File: my_robot_description/urdf/robot.urdf.xacro (robot description, xacro)
@@ -1,4 +1,5 @@
 <?xml version="1.0"?>
 <robot name="my_robot" xmlns:xacro="http://www.ros.org/wiki/xacro">
+     <xacro:include filename="$(find my_robot_description)/urdf/robot.gazebo.xacro"/>
     <xacro:property name="base_length" value="0.3"/>
     <xacro:property name="base_width"  value="0.3"/>
@@ -44,5 +45,5 @@
     <link name="lidar_link">
         <visual>
-            <geometry><mesh filename="$(dirname)/../meshes/lidar.STL"/></geometry>
+            <geometry><mesh filename="package://my_robot_description/meshes/lidar.STL"/></geometry>
             <material name="lidar_gray"><color rgba="0.5 0.5 0.5 1.0"/></material>
         </visual>
