Commit message: Update gazebo.launch.py and robot.urdf.xacro

File: my_robot_description/urdf/robot.urdf.xacro (robot description, xacro)
@@ -1,5 +1,6 @@
 <?xml version="1.0"?>
 <robot name="my_robot" xmlns:xacro="http://www.ros.org/wiki/xacro">
-     <xacro:include filename="$(find my_robot_description)/urdf/robot.gazebo.xacro"/>
+    <xacro:include filename="$(find my_robot_description)/urdf/robot.gazebo.xacro"/>
+    <xacro:arg name="mesh_path" default="package://my_robot_description/meshes/"/>
     <xacro:property name="base_length" value="0.3"/>
     <xacro:property name="base_width"  value="0.3"/>
@@ -16,5 +17,4 @@
     <xacro:property name="lidar_mass"   value="0.1"/>
     <xacro:property name="lidar_z_offset" value="0.13"/>
-    <xacro:property name="mesh_path" default="/root/workspaces/ros2_ws/src/task4-my_robot_description/my_robot_description/meshes"/>
     <xacro:property name="base_footprint_z" value="0.15"/>
     <link name="base_footprint"/>
@@ -45,5 +45,5 @@
     <link name="lidar_link">
         <visual>
-            <geometry><mesh filename="package://my_robot_description/meshes/lidar.STL"/></geometry>
+            <geometry><mesh filename="$(arg mesh_path)lidar.STL"/></geometry>
             <material name="lidar_gray"><color rgba="0.5 0.5 0.5 1.0"/></material>
         </visual>
